Commit message: update module 4

File: src/custom_robot_description/urdf/6_axis_robot.urdf (robot description, URDF)
Before this commit: robot custom_robot, 2 links, 1 joints
Links:
- removed link base_link
- removed link link1
- added link tool0
Joints:
- removed joint base_link__link1
- added joint link6__tool0: type fixed, parent link6, child tool0, origin xyz=0.0 0.0 0.02 rpy=0.0 0.0 0.0

Commit message: ros control tuning

File: src/custom_robot_description/urdf/6_axis_robot.urdf (robot description, URDF)
Before this commit: robot custom_robot, 1 links, 1 joints
Links:
- added link world
Joints:
- added joint fixed: type fixed, parent world, child base_link
- added joint link1__link2: type revolute, parent link1, child link2, origin xyz=0 0.07 0.055 rpy=0 0 0, axis 0 1 0, limit lower=-3.14159 upper=3.14159 effort=1000.0 velocity=0.5

File: src/custom_robot_description/urdf/custom_gripper.xacro (robot description, xacro)
@@ -2,8 +2,10 @@
 <robot xmlns:xacro="http://www.ros.org/wiki/xacro">
     <xacro:include filename="$(find custom_robot_description)/urdf/link_joint.xacro"/>
+    <xacro:include filename="$(find custom_robot_description)/urdf/6_axis_robot_gazebo.xacro"/>
     <!-- Model a gripper-->
     <xacro:macro name="custom_gripper" params = "parent origin_xyz" >
         <xacro:cobot_link_cylinder name="gripper_connector" origin_xyz="0.0 0.0 0.015" origin_rpy= "0 0 0"
-                            radius="0.04" length="0.03"  />
+                            radius="0.04" length="0.03" mass="0.5" i_xx="0.0002375" i_xy="0" i_xz="0"
+                            i_yy="0.0002375" i_yz="0" i_zz="0.00006666666667" />
         <joint name="{parent}__gripper_connector" type="fixed">
             <parent link="${parent}"/>
@@ -12,5 +14,6 @@
         </joint>
         <xacro:cobot_link_box name="finger_support" origin_xyz="0 0.005 0.005" origin_rpy="0 0 0"
-                                size="0.120 0.01 0.01" />
+                                size="0.120 0.01 0.01" mass="0.25" i_xx="0.0003" i_xy="0" i_xz="0"
+                            i_yy="0" i_yz="0" i_zz="0.0003"/>
         <joint name="finger_support__gripper_connector" type="fixed">
             <parent link="gripper_connector"/>
@@ -19,7 +22,9 @@
         </joint>
         <xacro:cobot_link_box name="finger_right" origin_xyz="0 0 0.04" origin_rpy="0 0 0"
-                                size="0.01 0.01 0.08" />
+                                size="0.01 0.01 0.08" mass="0.2" i_xx="0.00042667" i_xy="0" i_xz="0"
+                            i_yy="0" i_yz="0" i_zz="0.00042667"/>
         <xacro:cobot_link_box name="finger_left" origin_xyz="0 0 0.04" origin_rpy="0 0 0"
-                                size="0.01 0.01 0.08" />
+                                size="0.01 0.01 0.08" mass="0.2" i_xx="0.00042667" i_xy="0" i_xz="0"
+                            i_yy="0" i_yz="0" i_zz="0.00042667"/>
         <joint name="finger_right_joint" type="prismatic">
             <parent link="finger_support"/>
@@ -27,5 +32,5 @@
             <axis xyz="1 0 0"/>
             <limit lower="0" upper="0.044" velocity="0.5" effort="200"/>
-            <origin xyz="-0.05 0.0 0.01" rpy="0 0 0"/>
+            <origin xyz="-0.05 0.0 0.011" rpy="0 0 0"/>
             <dynamics damping="1" friction="2"/>
         </joint>
@@ -35,8 +40,16 @@
             <axis xyz="1 0 0"/>
             <limit lower="-0.044" upper="0" velocity="0.5" effort="200"/>
-            <origin xyz="0.05 0.0 0.01" rpy="0 0 0"/>
+            <origin xyz="0.05 0.0 0.011" rpy="0 0 0"/>
             <dynamics damping="1" friction="2"/>
             <mimic joint="finger_right_joint" multiplier="-1.0" offset="0" />
         </joint>
+        <xacro:transmission name="trans_finger_right_joint"
+                        joint_name="finger_right_joint"
+                        actuator_name="motor_finger_right_joint" />
+        <xacro:transmission name="trans_finger_left_joint"
+                        joint_name="finger_left_joint"
+                        actuator_name="motor_finger_left_joint" />
+        <xacro:mimic_joint_plugin_gazebo  parent_joint="finger_right_joint" mimic_joint="finger_left_joint"
+                                            has_pid="false" multiplier="-1.0" max_effort="200" />
     </xacro:macro>
 </robot>

File: src/custom_robot_description/urdf/link_joint.xacro (robot description, xacro)
@@ -1,6 +1,11 @@
 <?xml version = "1.0"?>
 <robot xmlns:xacro="http://www.ros.org/wiki/xacro">
-    <xacro:macro name="cobot_link_cylinder" params="name origin_xyz origin_rpy radius length">
+    <xacro:macro name="cobot_link_cylinder" params="name origin_xyz origin_rpy radius length mass i_xx i_xy i_xz i_yy i_yz i_zz">
         <link name="${name}">
+            <inertial>
+                <origin xyz="${origin_xyz}" rpy="${origin_rpy}"/>
+                <mass value="${mass}"/>
+                <inertia ixx="${i_xx}" ixy="${i_xy}" ixz="${i_xz}" iyy="${i_yy}" iyz="${i_yz}" izz="${i_zz}"/>
+            </inertial>
             <visual>
                 <geometry>
@@ -17,6 +22,11 @@
         </link>
     </xacro:macro>
-    <xacro:macro name="cobot_link_box" params="name origin_xyz origin_rpy size">
+    <xacro:macro name="cobot_link_box" params="name origin_xyz origin_rpy size mass i_xx i_xy i_xz i_yy i_yz i_zz">
         <link name="${name}">
+            <inertial>
+                <origin xyz="${origin_xyz}" rpy="${origin_rpy}"/>
+                <mass value="${mass}"/>
+                <inertia ixx="${i_xx}" ixy="${i_xy}" ixz="${i_xz}" iyy="${i_yy}" iyz="${i_yz}" izz="${i_zz}"/>
+            </inertial>
             <visual>
                 <geometry>
@@ -42,3 +52,15 @@
         </joint>
     </xacro:macro>
+    <xacro:macro name="transmission" params="name joint_name actuator_name">
+        <transmission name="${name}" >
+            <type>transmission_interface/SimpleTransmission</type>
+            <joint name = "${joint_name}" >
+                <hardwareInterface>hardware_interface/EffortJointInterface</hardwareInterface>
+            </joint>
+            <actuator name="${actuator_name}" >
+                <hardwareInterface>hardware_interface/EffortJointInterface</hardwareInterface>
+                <mechanicalReduction>1</mechanicalReduction>
+            </actuator>
+        </transmission>
+    </xacro:macro>
 </robot>
