Commit message: launch file in Gazebo pkg

File: src/custom_robot_description/urdf/custom_gripper.xacro (robot description, xacro)
@@ -35,5 +35,5 @@
             <dynamics damping="1" friction="2"/>
         </joint>
-        <xacro:transmission name="trans_finger_right_joint"
+        <xacro:transmission_effort name="trans_finger_right_joint"
                         joint_name="finger_right_joint"
                         actuator_name="motor_finger_right_joint" />
@@ -47,5 +47,5 @@
             <mimic joint="finger_right_joint" multiplier="-1.0" offset="0" />
         </joint>
-        <xacro:transmission name="trans_finger_left_joint"
+        <xacro:transmission_effort name="trans_finger_left_joint"
                         joint_name="finger_left_joint"
                         actuator_name="motor_finger_left_joint" />

File: src/custom_robot_description/urdf/link_joint.xacro (robot description, xacro)
@@ -56,4 +56,16 @@
             <type>transmission_interface/SimpleTransmission</type>
             <joint name = "${joint_name}" >
+                <hardwareInterface>hardware_interface/PositionJointInterface</hardwareInterface>
+            </joint>
+            <actuator name="${actuator_name}" >
+                <hardwareInterface>hardware_interface/PositionJointInterface</hardwareInterface>
+                <mechanicalReduction>1</mechanicalReduction>
+            </actuator>
+        </transmission>
+    </xacro:macro>
+    <xacro:macro name="transmission_effort" params="name joint_name actuator_name">
+        <transmission name="${name}" >
+            <type>transmission_interface/SimpleTransmission</type>
+            <joint name = "${joint_name}" >
                 <hardwareInterface>hardware_interface/EffortJointInterface</hardwareInterface>
             </joint>
