Commit message: add jointTrajectoryController

File: src/ur5_description/urdf/ur5_gripper.xacro (robot description, xacro)
@@ -17,3 +17,15 @@
   <xacro:include filename="$(find ur5_description)/urdf/eef.xacro"/>
   <xacro:ur5_robot prefix="" />
+  <link name="world">
+  </link>
+  <joint name="fixed" type="fixed">
+        <parent link="world"/>
+        <child link="base_link"/>
+  </joint>
+    <gazebo>
+      <plugin name="ros_control" filename="libgazebo_ros_control.so">
+        <robotNamespace>/ur5</robotNamespace>
+        <!-- <robotSimType>gazebo_ros_control/DefaultRobotHWSim</robotSimType> -->
+      </plugin>
+    </gazebo>
 </robot>

Commit message: update ur5 moveit config

File: src/ur5_description/urdf/ur5_gripper.xacro (robot description, xacro)
@@ -22,4 +22,5 @@
         <parent link="world"/>
         <child link="base_link"/>
+        <origin xyz="0 0.0 0.8" rpy="0 0 0"/>
   </joint>
     <gazebo>
